File: manufacturing/STM32_DevBoard/RevHist.kicad_sch (KiCad schematic)
At the start: 0 parts

Commit message: upd Schematic
Other:
- company: (none) -> s-grundner
- title: (none) -> STM32-DevBoard
Changed lines of the file:
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@@
 (kicad_sch (version 20230121) (generator eeschema)
   (paper "A4")
+  (title_block
+    (title "STM32-DevBoard")
+    (date "2023-08-20")
+    (rev "R0")
+    (company "s-grundner")
+  )
 )
