File: manufacturing/STM32_DevBoard/STM32_DevBoard.kicad_sch (KiCad schematic)
At the start: 0 parts

Commit message: upd Schematic
Other:
- sheet Connectors ports: added A_GPIO_0, A_GPIO_1, A_GPIO_2, A_GPIO_3, A_GPIO_4, A_GPIO_5, A_GPIO_6, A_GPIO_7, CAN_RX, CAN_TX, I2C_SCL, I2C_SDA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; removed none
- sheet MCU ports: added A_GPIO_0, A_GPIO_1, A_GPIO_2, A_GPIO_3, A_GPIO_4, A_GPIO_5, A_GPIO_6, A_GPIO_7, CAN_RX, CAN_TX, I2C_SCL, I2C_SDA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; removed none
- sheet Sensors ports: added IMU_INT, SENSE_SCL, SENSE_SDA; removed none
- note removed: "Power"
