File: manufacturing/STM32_DevBoard/CONN.kicad_sch (KiCad schematic)
At the start: 0 parts

Commit message: upd Schematic
Parts:
- added C1 (x4): 100n, Capacitor_SMD:C_0805_2012Metric_Pad1.18x1.45mm_HandSolder, symbol Device:C_Small
- added C1: 100n, Capacitor_SMD:C_0805_2012Metric_Pad1.18x1.45mm_HandSolder, symbol Device:C
- added C23, C25: 560n, Capacitor_SMD:C_0805_2012Metric_Pad1.18x1.45mm_HandSolder, symbol Device:C_Small
- added C6: 2u2, Capacitor_SMD:C_0805_2012Metric_Pad1.18x1.45mm_HandSolder, symbol Device:C_Small
- added D10, D11, D12, D13, D14, D16, D17, D18, D19, D22, D23, D3, D4, D7, D8, D9: 3V3, Diode_SMD:D_SOD-923, symbol Diode:ESD9B3.3ST5G
- added J1: CAN, Connector_Molex:Molex_Micro-Latch_53254-0470_1x04_P2.00mm_Horizontal, symbol Connector:Conn_01x04_Pin
- added J10: I2C, Connector_Molex:Molex_Micro-Latch_53254-0470_1x04_P2.00mm_Horizontal, symbol Connector:Conn_01x04_Pin
- added J11: PWM0, Connector_Molex:Molex_Micro-Latch_53254-0370_1x03_P2.00mm_Horizontal, symbol Connector:Conn_01x03_Pin
- added J12, J3: Conn_01x03_Pin, Connector_Molex:Molex_Micro-Latch_53254-0370_1x03_P2.00mm_Horizontal, symbol Connector:Conn_01x03_Pin
- added J5: USB_A, Connector_USB:USB_A_CONNFLY_DS1095-WNR0, symbol Connector:USB_A
- added J8: SPI/UART, Connector_Molex:Molex_Micro-Latch_53254-0570_1x05_P2.00mm_Horizontal, symbol Connector:Conn_01x05_Pin
- added J9: SPI_NSS/GPIO, Connector_PinHeader_2.54mm:PinHeader_1x03_P2.54mm_Vertical, symbol Connector:Conn_01x03_Pin
- added R1 (x2): 47R, Resistor_SMD:R_0805_2012Metric_Pad1.20x1.40mm_HandSolder, symbol Device:R
- added R1 (x2): 56R, Resistor_SMD:R_0805_2012Metric_Pad1.20x1.40mm_HandSolder, symbol Device:R_Small
- added R10: 5k6, Resistor_SMD:R_0805_2012Metric_Pad1.20x1.40mm_HandSolder, symbol Device:R
- added R10, R12: 150R, Resistor_SMD:R_0805_2012Metric_Pad1.20x1.40mm_HandSolder, symbol Device:R_Small
- added R18, R19, R20, R21, R22, R7: 10R, Resistor_SMD:R_0805_2012Metric_Pad1.20x1.40mm_HandSolder, symbol Device:R_Small
- added U3: SN65HVD230, Package_SO:SOIC-8_3.9x4.9mm_P1.27mm, symbol Interface_CAN_LIN:SN65HVD230
- added U4 (x2): USBLC6-2, Package_TO_SOT_SMD:SOT-23-6, symbol Power_Protection:WE-TVS-82400102
Connections:
- new net: D18.2 (A2), J10.2 (Pin_2), R22.2
- new net: D12.2 (A2), J9.1 (Pin_1), R18.2
- new net: R1.2, U3.1 (D)
- new net: R1.2, U3.4 (R)
- new net: D9.2 (A2), J8.4 (Pin_4), R7.2
- new net: D7.2 (A2), J3.2 (Pin_2), R10.2
- new net: D22.2 (A2), J12.2 (Pin_2), R12.2
- new net: D11.2 (A2), J9.2 (Pin_2), R19.2
- new net: D10.2 (A2), J9.3 (Pin_3), R20.2
- new net: D8.2 (A2), J8.3 (Pin_3), R21.2
- new net +3V3: C1.1, C6.1, D14.2 (A2), D16.2 (A2), D19.2 (A2), D23.2 (A2), D3.2 (A2), J1.1 (Pin_1), J10.1 (Pin_1), J11.1 (Pin_1), J12.1 (Pin_1), J3.1 (Pin_1), J8.1 (Pin_1), U3.3 (VCC), U4.5
- new net +5V: J5.1 (VBUS), U4.5
- new net A_GPIO_0: C25.1, R12.1
- new net A_GPIO_1: C23.1, R10.1
- new net CAN+: C1.1, R1.2, U3.7 (CANH), U4.1
- new net CAN-: C1.2, R1.1, U3.6 (CANL), U4.3
- new net CAN_CONN+: J1.2 (Pin_2), U4.6
- new net CAN_CONN-: J1.3 (Pin_3), U4.4
- new net CAN_RS: C1.1, R10.2, U3.8 (Rs)
- new net CAN_RX: R1.1
- new net CAN_TX: R1.1
- new net GND: C1.1, C1.2, C1.2, C1.2, C1.2, C23.2, C25.2, C6.2, D10.1 (A1), D11.1 (A1), D12.1 (A1), D13.1 (A1), D14.1 (A1), D16.1 (A1), D17.1 (A1), D18.1 (A1), D19.1 (A1), D22.1 (A1), D23.1 (A1), D3.1 (A1), D4.1 (A1), D7.1 (A1), D8.1 (A1), D9.1 (A1), J1.4 (Pin_4), J10.4 (Pin_4), J11.3 (Pin_3), J12.3 (Pin_3), J3.3 (Pin_3), J5.4 (GND), J8.5 (Pin_5), R10.1, U3.2 (GND), U4.2, U4.2
- new net I2C_SCL: R22.1
- new net I2C_SDA: D17.2 (A2), J10.3 (Pin_3)
- new net PWM0: D13.2 (A2), J11.2 (Pin_2)
- new net SPI_MISO_RX: R21.1
- new net SPI_MOSI: D4.2 (A2), J8.2 (Pin_2)
- new net SPI_NSS0: R18.1
- new net SPI_NSS1: R19.1
- new net SPI_NSS2: R20.1
- new net SPI_SCK_TX: R7.1
- new net USB_CONN+: J5.3 (D+), U4.6
- new net USB_CONN-: J5.2 (D-), U4.4
- new net USB_D+: U4.1
- new net USB_D-: U4.3
- new net VREF: C1.1, R1.1, R1.2, U3.5 (Vref)
- no-connect marks 0 -> 1
Other:
- note added: "Analog GPIOS"
- note added: "CAN Interface"
- note added: "CAN RS Pin Config (Mode Select):"
- note added: "Connectors"
- note added: "I2C"
- note added: "PWM"
- note added: "SPI/UART"
- note added: "Strong Pulldown -> High Speed Strong Pullup -> Low Power 10k-100k Pulldown -> Slope Control"
- note added: "USB"
- company: (none) -> s-grundner
- title: (none) -> STM32-DevBoard

Commit message: update Board Revision 0
Parts:
- removed D14, D16, D19, D23: 3V3, Diode_SMD:D_SOD-923, symbol Diode:ESD9B3.3ST5G
- removed U4 (x2): USBLC6-2, Package_TO_SOT_SMD:SOT-23-6, symbol Power_Protection:WE-TVS-82400102
- added D15, D20, D5, D6: 3V3, Diode_SMD:D_SOD-923, symbol Diode:ESD9B3.3ST5G
- added D2: GN, LED_THT:LED_D3.0mm, symbol Device:LED
- added R11: 1k5, Resistor_SMD:R_0805_2012Metric_Pad1.20x1.40mm_HandSolder, symbol Device:R_Small
- added R17: 10R, Resistor_SMD:R_0805_2012Metric_Pad1.20x1.40mm_HandSolder, symbol Device:R_Small
- J11: footprint Connector_Molex:Molex_Micro-Latch_53254-0370_1x03_P2.00mm_Horizontal -> Connector_PinHeader_2.54mm:PinHeader_1x03_P2.54mm_Vertical
- J12, J3: value Conn_01x03_Pin -> AGPIO; footprint Connector_Molex:Molex_Micro-Latch_53254-0370_1x03_P2.00mm_Horizontal -> Connector_PinHeader_2.54mm:PinHeader_1x03_P2.54mm_Vertical
- U3: LCSC (none) -> C12084
Connections:
- net CAN_CONN+ is gone; now on net CAN+: J1.2 (Pin_2)
- net CAN_CONN- is gone; now on net CAN-: J1.3 (Pin_3)
- net USB_CONN+ is gone; now on net USB_D+: J5.3 (D+)
- net USB_CONN- is gone; now on net USB_D-: J5.2 (D-)
- net +3V3: now also R11.2
- net CAN+: now also D20.2 (A2)
- net CAN-: now also D15.2 (A2)
- net GND: now also D15.1 (A1), D2.1 (K), D20.1 (A1), D5.1 (A1), D6.1 (A1)
- net PWM0: now also R17.1; no longer D13.2 (A2), J11.2 (Pin_2)
- net USB_D+: now also D5.2 (A2)
- net USB_D-: now also D6.2 (A2)
- net A_GPIO_0 renamed A_GPIO_2
- net A_GPIO_1 renamed A_GPIO_3
- new net: D2.2 (A), R11.1
- new net: D13.2 (A2), J11.2 (Pin_2), R17.2
Other:
- moved on the sheet: C23, C25, D13, D17, D18, D22, D7, J1, J10, J11, J12, J3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
