File: manufacturing/STM32_DevBoard/MCU.kicad_sch (KiCad schematic)
At the start: 13 parts, among them U3 STM32F405RGT6, U4 CAT24C256

Commit message: upd Schematic
Parts:
- added C18: 100n, Capacitor_SMD:C_0805_2012Metric_Pad1.18x1.45mm_HandSolder, symbol Device:C_Small
- added D1: LED_RGBA, LED_SMD:LED_SK6812MINI_PLCC4_3.5x3.5mm_P1.75mm, symbol Device:LED_RGBA
- added J6: SWD, Connector_PinHeader_2.54mm:PinHeader_2x05_P2.54mm_Vertical, symbol Connector_Generic:Conn_02x05_Odd_Even
- added R2: 10k, Resistor_SMD:R_0805_2012Metric_Pad1.20x1.40mm_HandSolder, symbol Device:R
- added R23, R24, R25, R26, R27, R28, R4, R5, R6: 1k5, Resistor_SMD:R_0805_2012Metric_Pad1.20x1.40mm_HandSolder, symbol Device:R
- added SW1: EEPROM_WP, Button_Switch_THT:SW_E-Switch_EG1271_SPDT, symbol Switch:SW_SPDT
- C10, C9: value C -> 2u2; footprint (none) -> Capacitor_SMD:C_0805_2012Metric_Pad1.18x1.45mm_HandSolder
- U4: value CAT24C256 -> AT24C256; footprint (none) -> Package_SO:SOIC-8_3.9x4.9mm_P1.27mm; LCSC (none) -> C6482
Connections:
- net +3V3: now also C8.1, FB1.2, U4.8 (VCC), C18.1, D1.4 (A), J6.1 (Pin_1), R23.1, R24.1, R25.1, R26.1, R27.1, R28.1, SW1.1 (A); no longer C7.1, FB1.1, U3.13 (VDDA)
- net GND: now also C1.2, C2.2, C3.2, C4.2, C5.2, C6.2, U4.1 (A0), U4.2 (A1), U4.3 (A2), U4.4 (GND), C18.2, J6.3 (Pin_3), J6.5 (Pin_5), J6.9 (Pin_9), SW1.3 (C)
- net A_GPIO_0: now reaches U3.14 (PA0)
- net A_GPIO_1: now reaches U3.15 (PA1)
- net A_GPIO_2: now reaches U3.16 (PA2)
- net A_GPIO_3: now reaches U3.17 (PA3)
- net A_GPIO_4: now reaches U3.20 (PA4)
- net A_GPIO_5: now reaches U3.21 (PA5)
- net A_GPIO_6: now reaches U3.22 (PA6)
- net A_GPIO_7: now reaches U3.23 (PA7)
- net PWM0: now reaches U3.26 (PB0)
- net PWM1: now reaches U3.27 (PB1)
- net I2C_SCL: now reaches U3.29 (PB10)
- net I2C_SCL: now also R27.2
- net I2C_SDA: now reaches U3.30 (PB11)
- net I2C_SDA: now also R28.2
- net CAN_RX: now reaches U3.33 (PB12)
- net CAN_TX: now reaches U3.34 (PB13)
- net SENSE_SDA: now reaches U3.40 (PC9)
- net SENSE_SDA: now also R26.2
- net SENSE_SCL: now reaches U3.41 (PA8)
- net SENSE_SCL: now also R25.2
- net IMU_INT: now reaches U3.42 (PA9)
- net USB_D-: now reaches U3.44 (PA11)
- net USB_D+: now reaches U3.45 (PA12)
- net SWDIO: now reaches U3.46 (PA13)
- net SWDIO: now also J6.2 (Pin_2)
- net SWCLK: now reaches U3.49 (PA14)
- net SWCLK: now also J6.4 (Pin_4)
- net SPI_NSS0: now reaches U3.50 (PA15)
- net SPI_SCK_TX: now reaches U3.51 (PC10)
- net SPI_MISO_RX: now reaches U3.52 (PC11)
- net SPI_MOSI: now reaches U3.53 (PC12)
- net SPI_NSS1: now reaches U3.54 (PD2)
- net SWO: now reaches U3.55 (PB3)
- net SWO: now also J6.6 (Pin_6)
- net SPI_NSS2: now reaches U3.56 (PB4)
- net NPWM_B: now reaches U3.57 (PB5)
- net NPWM_B: now also R6.1
- net NPWM_G: now reaches U3.58 (PB6)
- net NPWM_G: now also R5.1
- net NPWM_R: now reaches U3.59 (PB7)
- net NPWM_R: now also R4.1
- net EEPROM_SCL: now reaches U3.61 (PB8)
- net EEPROM_SCL: now also U4.6 (SCL), R24.2
- net EEPROM_SDA: now reaches U3.62 (PB9)
- net EEPROM_SDA: now also U4.5 (SDA), R23.2
- net EEPROM_WP: now reaches U4.7 (WP)
- net EEPROM_WP: now also R2.2
- net Strapping/NRST renamed NRST
- net NRST: now also J6.10 (Pin_10)
- new net: D1.1 (RK), R4.2
- new net: D1.3 (BK), R6.2
- new net: D1.2 (GK), R5.2
- new net +3V3A: C7.1, FB1.1, U3.13 (VDDA)
- new net EEPROM_WP_SW: R2.1, SW1.2 (B)
- no-connect marks 0 -> 18
Other:
- company: (none) -> s-grundner
- title: (none) -> STM32-DevBoard
- moved on the sheet: C10, C8, C9, U4

Commit message: update Board Revision 0
Parts:
- FB1: value xR @ xMHz -> 100R @ 100MHz; LCSC (none) -> C1015
- U3: LCSC (none) -> C15742
Changed lines of the file:
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@@
+      (effects (font (size 1.27 1.27)) hide)
+    )
+    (property "LCSC" "C15742" (at 101.6 91.44 0)
       (effects (font (size 1.27 1.27)) hide)
     )
@@
       (effects (font (size 1.27 1.27)))
     )
-    (property "Value" "xR @ xMHz" (at 129.5019 29.21 90)
+    (property "Value" "100R @ 100MHz" (at 129.5019 29.21 90)
       (effects (font (size 1.27 1.27)))
     )
@@
       (effects (font (size 1.27 1.27)) hide)
     )
+    (property "LCSC" "C1015" (at 129.54 33.02 0)
+      (effects (font (size 1.27 1.27)) hide)
+    )
