File: manufacturing/STM32_DevBoard/MCU_Strapping.kicad_sch (KiCad schematic)
At the start: 10 parts, among them SW1 SW_SPDT, SW2 SW_Omron_B3FS, Y1 25MHz

Commit message: upd Schematic
Parts:
- removed C14: C, symbol Device:C
- C11, C12: footprint (none) -> Capacitor_SMD:C_0805_2012Metric_Pad1.18x1.45mm_HandSolder
- C13: value C -> 820n; footprint (none) -> Capacitor_SMD:C_0805_2012Metric_Pad1.18x1.45mm_HandSolder
- R1, R3: footprint (none) -> Resistor_SMD:R_0805_2012Metric_Pad1.20x1.40mm_HandSolder
- R2: value R -> 10k; footprint (none) -> Resistor_SMD:R_0805_2012Metric_Pad1.20x1.40mm_HandSolder
- SW1: footprint (none) -> Button_Switch_THT:SW_E-Switch_EG1271_SPDT
- SW2: footprint (none) -> Button_Switch_THT:SW_PUSH_6mm
- Y1: value 25MHz -> 25MHz 12pF; footprint (none) -> Crystal:Crystal_SMD_3225-4Pin_3.2x2.5mm; LCSC (none) -> C9006
Other:
- company: (none) -> s-grundner
- title: (none) -> STM32-DevBoard
Changed lines of the file:
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@@
 (kicad_sch (version 20230121) (generator eeschema)
   (paper "A4")
-  (junction (at 185.42 107.95) (diameter 0) (color 0 0 0 0)
+  (title_block
+    (title "STM32-DevBoard")
+    (date "2023-08-20")
+    (rev "R0")
+    (company "s-grundner")
   )
   (junction (at 201.93 99.06) (diameter 0) (color 0 0 0 0)
   )
-  (junction (at 196.85 99.06) (diameter 0) (color 0 0 0 0)
-  )
   (junction (at 86.36 101.6) (diameter 0) (color 0 0 0 0)
   )
@@
     (stroke (width 0) (type default))
   )
-  (wire (pts (xy 185.42 99.06) (xy 185.42 107.95))
+  (wire (pts (xy 185.42 99.06) (xy 185.42 109.22))
     (stroke (width 0) (type default))
   )
@@
     (stroke (width 0) (type default))
   )
-  (wire (pts (xy 196.85 99.06) (xy 196.85 107.95))
-    (stroke (width 0) (type default))
-  )
   (wire (pts (xy 96.52 107.95) (xy 96.52 106.68))
     (stroke (width 0) (type default))
   )
-  (wire (pts (xy 196.85 99.06) (xy 201.93 99.06))
+  (wire (pts (xy 195.58 99.06) (xy 201.93 99.06))
     (stroke (width 0) (type default))
   )
@@
     (stroke (width 0) (type default))
   )
-  (wire (pts (xy 196.85 107.95) (xy 194.31 107.95))
-    (stroke (width 0) (type default))
-  )
-  (wire (pts (xy 185.42 107.95) (xy 185.42 109.22))
-    (stroke (width 0) (type default))
-  )
-  (wire (pts (xy 195.58 99.06) (xy 196.85 99.06))
-    (stroke (width 0) (type default))
-  )
   (wire (pts (xy 95.25 107.95) (xy 95.25 114.3))
     (stroke (width 0) (type default))
@@
   )
   (wire (pts (xy 86.36 101.6) (xy 90.17 101.6))
-    (stroke (width 0) (type default))
-  )
-  (wire (pts (xy 185.42 107.95) (xy 186.69 107.95))
     (stroke (width 0) (type default))
   )
@@
       (effects (font (size 1.27 1.27)))
     )
-    (property "Value" "R" (at 148.59 99.06 90)
-      (effects (font (size 1.27 1.27)))
-    )
-    (property "Footprint" "" (at 148.59 103.378 90)
+    (property "Value" "10k" (at 148.59 99.06 90)
+      (effects (font (size 1.27 1.27)))
+    )
+    (property "Footprint" "Resistor_SMD:R_0805_2012Metric_Pad1.20x1.40mm_HandSolder" (at 148.59 103.378 90)
       (effects (font (size 1.27 1.27)) hide)
     )
@@
       (effects (font (size 1.27 1.27)))
     )
-    (property "Footprint" "" (at 138.43 101.6 0)
+    (property "Footprint" "Button_Switch_THT:SW_E-Switch_EG1271_SPDT" (at 138.43 101.6 0)
       (effects (font (size 1.27 1.27)) hide)
     )
@@
       (effects (font (size 1.27 1.27)) (justify left))
     )
-    (property "Footprint" "" (at 200.152 93.98 90)
+    (property "Footprint" "Resistor_SMD:R_0805_2012Metric_Pad1.20x1.40mm_HandSolder" (at 200.152 93.98 90)
       (effects (font (size 1.27 1.27)) hide)
     )
@@
       (effects (font (size 1.27 1.27)) (justify left))
     )
-    (property "Footprint" "" (at 87.3252 113.03 0)
+    (property "Footprint" "Capacitor_SMD:C_0805_2012Metric_Pad1.18x1.45mm_HandSolder" (at 87.3252 113.03 0)
       (effects (font (size 1.27 1.27)) hide)
     )
@@
       (effects (font (size 1.27 1.27)))
     )
-    (property "Footprint" "" (at 190.5 93.98 0)
+    (property "Footprint" "Button_Switch_THT:SW_PUSH_6mm" (at 190.5 93.98 0)
       (effects (font (size 1.27 1.27)) hide)
     )
@@
       (effects (font (size 1.27 1.27)) (justify left))
     )
-    (property "Value" "C" (at 205.74 105.41 0)
-      (effects (font (size 1.27 1.27)) (justify left))
-    )
-    (property "Footprint" "" (at 202.8952 107.95 0)
+    (property "Value" "820n" (at 205.74 105.41 0)
+      (effects (font (size 1.27 1.27)) (justify left))
+    )
+    (property "Footprint" "Capacitor_SMD:C_0805_2012Metric_Pad1.18x1.45mm_HandSolder" (at 202.8952 107.95 0)
       (effects (font (size 1.27 1.27)) hide)
     )
@@
       (effects (font (size 1.27 1.27)))
     )
-    (property "Footprint" "" (at 105.918 96.52 90)
+    (property "Footprint" "Resistor_SMD:R_0805_2012Metric_Pad1.20x1.40mm_HandSolder" (at 105.918 96.52 90)
       (effects (font (size 1.27 1.27)) hide)
     )
@@
         (path "/936a9920-4479-4b68-af43-551df89037a4/4885c666-6066-41ae-b6bc-46cba658e96a/3468291a-9e84-495b-9f59-5c9432283e7c"
           (reference "#PWR010") (unit 1)
-        )
-      )
-    )
-  )
-  (symbol (lib_id "Device:C") (at 190.5 107.95 270) (unit 1)
-    (in_bom yes) (on_board yes) (dnp no)
-    (property "Reference" "C14" (at 190.5 101.6 90)
-      (effects (font (size 1.27 1.27)))
-    )
-    (property "Value" "C" (at 190.5 104.14 90)
-      (effects (font (size 1.27 1.27)))
-    )
-    (property "Footprint" "" (at 186.69 108.9152 0)
-      (effects (font (size 1.27 1.27)) hide)
-    )
-    (property "Datasheet" "~" (at 190.5 107.95 0)
-      (effects (font (size 1.27 1.27)) hide)
-    )
-    (pin "1")
-    (pin "2")
-    (instances
-      (project "STM32_DevBoard"
-        (path "/936a9920-4479-4b68-af43-551df89037a4/4885c666-6066-41ae-b6bc-46cba658e96a/3468291a-9e84-495b-9f59-5c9432283e7c"
-          (reference "C14") (unit 1)
         )
       )
@@
       (effects (font (size 1.27 1.27)))
     )
-    (property "Value" "25MHz" (at 95.25 96.52 0)
-      (effects (font (size 1.27 1.27)))
-    )
-    (property "Footprint" "" (at 95.25 101.6 0)
-      (effects (font (size 1.27 1.27)) hide)
-    )
-    (property "Datasheet" "~" (at 95.25 101.6 0)
+    (property "Value" "25MHz 12pF" (at 95.25 96.52 0)
+      (effects (font (size 1.27 1.27)))
+    )
+    (property "Footprint" "Crystal:Crystal_SMD_3225-4Pin_3.2x2.5mm" (at 95.25 101.6 0)
+      (effects (font (size 1.27 1.27)) hide)
+    )
+    (property "Datasheet" "https://datasheet.lcsc.com/lcsc/2304140030_Yangxing-Tech-X322525MOB4SI_C9006.pdf" (at 95.25 101.6 0)
+      (effects (font (size 1.27 1.27)) hide)
+    )
+    (property "LCSC" "C9006" (at 95.25 101.6 0)
       (effects (font (size 1.27 1.27)) hide)
     )
@@
       (effects (font (size 1.27 1.27)) (justify left))
     )
-    (property "Footprint" "" (at 105.1052 113.03 0)
-      (effects (font (size 1.27 1.27)) hide)
-    )
+    (property "Footprint" "Capacitor_SMD:C_0805_2012Metric_Pad1.18x1.45mm_HandSolder" (at 105.1052 113.03 0)
+      (effects (font (size 1.27 1.27)) hide)
+    )

Commit message: update Board Revision 0
Parts:
- C11, C12: value C -> 12p
- R1: value R -> 0R
- R3: value R -> 10k
Changed lines of the file:
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@@
       (effects (font (size 1.27 1.27)) (justify left))
     )
-    (property "Value" "R" (at 204.47 95.25 0)
+    (property "Value" "10k" (at 204.47 95.25 0)
       (effects (font (size 1.27 1.27)) (justify left))
     )
@@
       (effects (font (size 1.27 1.27)) (justify left))
     )
-    (property "Value" "C" (at 88.9 110.49 0)
+    (property "Value" "12p" (at 88.9 110.49 0)
       (effects (font (size 1.27 1.27)) (justify left))
     )
@@
       (effects (font (size 1.27 1.27)))
     )
-    (property "Value" "R" (at 106.68 97.79 0)
+    (property "Value" "0R" (at 106.68 97.79 0)
       (effects (font (size 1.27 1.27)))
     )
@@
       (effects (font (size 1.27 1.27)) (justify left))
     )
-    (property "Value" "C" (at 106.68 110.49 0)
-      (effects (font (size 1.27 1.27)) (justify left))
-    )
+    (property "Value" "12p" (at 106.68 110.49 0)
+      (effects (font (size 1.27 1.27)) (justify left))
+    )
