File: manufacturing/STM32_DevBoard/PMU.kicad_sch (KiCad schematic)
At the start: 0 parts

Commit message: upd Schematic
Parts:
- added C22, C6: 2u2, Capacitor_SMD:C_0805_2012Metric_Pad1.18x1.45mm_HandSolder, symbol Device:C
- added C4: 100n, Capacitor_SMD:C_0805_2012Metric_Pad1.18x1.45mm_HandSolder, symbol Device:C
- added C6: 10u, Capacitor_SMD:C_0805_2012Metric_Pad1.18x1.45mm_HandSolder, symbol Device:C
- added D2: B5819W, Diode_SMD:D_SOD-123, symbol Device:D_Schottky
- added FB1: xR @ xMHz, Inductor_SMD:L_0805_2012Metric_Pad1.05x1.20mm_HandSolder, symbol Device:FerriteBead_Small
- added L1: 3u3, Inductor_SMD:L_7.3x7.3_H4.5, symbol Device:L
- added U2: LMR16006YQ3, Package_TO_SOT_SMD:SOT-23-6, symbol Regulator_Switching:LMR16006YQ3
Connections:
- new net +3V3: C6.1, L1.2, U2.3 (FB)
- new net +5V: D2.2 (A)
- new net BUCK_BST: C4.1, U2.1 (CB)
- new net BUCK_IN: C6.1, FB1.1, U2.4 (~{SHDN}), U2.5 (VIN)
- new net BUCK_OUT: C4.2, L1.1, U2.6 (SW)
- new net GND: C22.2, C6.2, C6.2, U2.2 (GND)
- new net POST_POL: C22.1, D2.1 (K), FB1.2
Other:
- company: (none) -> s-grundner
- title: (none) -> STM32-DevBoard

Commit message: update Board Revision 0
Parts:
- removed C4: 100n, Capacitor_SMD:C_0805_2012Metric_Pad1.18x1.45mm_HandSolder, symbol Device:C
- removed C6: 10u, Capacitor_SMD:C_0805_2012Metric_Pad1.18x1.45mm_HandSolder, symbol Device:C
- removed L1: 3u3, Inductor_SMD:L_7.3x7.3_H4.5, symbol Device:L
- removed U2: LMR16006YQ3, Package_TO_SOT_SMD:SOT-23-6, symbol Regulator_Switching:LMR16006YQ3
- added C14: 22u, Capacitor_THT:C_Radial_D5.0mm_H7.0mm_P2.00mm, symbol Device:C_Polarized
- added U8: AMS1117-3.3, Package_TO_SOT_SMD:SOT-223-3_TabPin2, symbol Regulator_Linear:AMS1117-3.3
- D2: LCSC (none) -> C8598
- FB1: value xR @ xMHz -> 100R @ 100MHz; LCSC (none) -> C1015
Connections:
- net +3V3: now also C14.1, U8.2 (VO)
- net GND: now also C14.2, U8.1 (GND)
- net BUCK_IN renamed LDO_IN
- net LDO_IN: now also U8.3 (VI)
