File: manufacturing/STM32_DevBoard/Sensors.kicad_sch (KiCad schematic)
At the start: 8 parts, among them U1 MPU-6050, U2 SHTC3

Commit message: upd Schematic
Parts:
- removed C18: 2u2, symbol Device:C
- C15, C16, C17, C20: footprint (none) -> Capacitor_SMD:C_0805_2012Metric_Pad1.18x1.45mm_HandSolder
- C19: value 100n -> 10n; footprint (none) -> Capacitor_SMD:C_0805_2012Metric_Pad1.18x1.45mm_HandSolder
Connections:
- net SENSE_SCL: now reaches U1.23 (SCL)
- net SENSE_SDA: now reaches U1.24 (SDA)
- net AUX_SCL: now reaches U1.6 (AUX_DA), U2.2 (SCL)
- net AUX_SDA: now reaches U1.7 (AUX_CL), U2.3 (SDA)
Other:
- company: (none) -> s-grundner
- title: (none) -> STM32-DevBoard
- moved on the sheet: C19

Commit message: update Board Revision 0
Parts:
- U1: LCSC (none) -> C24112
- U2: LCSC (none) -> C194656
Changed lines of the file:
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@@
+      (effects (font (size 1.27 1.27)) hide)
+    )
+    (property "LCSC" "C24112" (at 114.3 85.09 0)
       (effects (font (size 1.27 1.27)) hide)
     )
@@
       (effects (font (size 1.27 1.27)) hide)
     )
+    (property "LCSC" "C194656" (at 152.4 83.82 0)
+      (effects (font (size 1.27 1.27)) hide)
+    )
